Commit message: adding mapping feature

File: diff_bot/urdf/robot.urdf.xacro (robot description, xacro)
@@ -11,3 +11,9 @@
     <!-- Base Link -->
     <link name="base_link"/>
+    <!-- Base Footprint Link -->
+    <link name="base_footprint"/>
+    <joint name="base_footprint_joint" type="fixed">
+        <parent link="base_link"/>
+        <child link="base_footprint"/>
+    </joint>
 </robot>
